File: Adapter-IO4-Breakout.brd (EAGLE design)
At the start: 50 x 50 mm, 7 parts

Commit message: added values for connectors
Parts:
- CON1, CON2: value (none) -> RJ12/6
- GND, J3, V+: value (none) -> 0.100
Changed lines of the file:
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@@
 <elements>
 <element name="U$1" library="SparkFun" package="OSHW-LOGO-M" value="OSHW-LOGOM" x="43.18" y="42.926"/>
-<element name="J3" library="SPCoast" package="1X06_LOCK" value="" x="31.75" y="6.35" smashed="yes" rot="R180">
+<element name="J3" library="SPCoast" package="1X06_LOCK" value="0.100" x="31.75" y="6.35" smashed="yes" rot="R180">
 <attribute name="NAME" x="27.94" y="-0.508" size="1.27" layer="25" font="vector" rot="R180"/>
 <attribute name="VALUE" x="33.02" y="9.652" size="1.27" layer="27" font="vector" rot="R180"/>
 </element>
 <element name="BOARD1" library="SPCoast" package="BOARD-SEED5X5-NOHOLES" value="BOARD50X50-HOHOLES" x="0" y="0"/>
-<element name="V+" library="SPCoast" package="1X02_LOCK" value="" x="41.91" y="6.35" smashed="yes" rot="R90">
+<element name="V+" library="SPCoast" package="1X02_LOCK" value="0.100" x="41.91" y="6.35" smashed="yes" rot="R90">
 <attribute name="NAME" x="43.0022" y="12.6492" size="1.27" layer="25" ratio="10" rot="R180"/>
 <attribute name="VALUE" x="45.085" y="5.08" size="1.27" layer="27" rot="R90"/>
 </element>
-<element name="GND" library="SPCoast" package="1X02_LOCK" value="" x="8.89" y="6.35" smashed="yes" rot="R90">
+<element name="GND" library="SPCoast" package="1X02_LOCK" value="0.100" x="8.89" y="6.35" smashed="yes" rot="R90">
 <attribute name="NAME" x="10.9982" y="12.9032" size="1.27" layer="25" ratio="10" rot="R180"/>
 <attribute name="VALUE" x="12.065" y="5.08" size="1.27" layer="27" rot="R90"/>
 </element>
-<element name="CON1" library="SPCoast" package="RJ25-PANEL" value="" x="45.72" y="25.4" rot="R90">
+<element name="CON1" library="SPCoast" package="RJ25-PANEL" value="RJ12/6" x="45.72" y="25.4" rot="R90">
 <attribute name="AMP" value="520250-3" x="45.72" y="25.4" size="1.778" layer="27" font="vector" ratio="10" rot="R90" display="off"/>
 <attribute name="OPL" value="none" x="45.72" y="25.4" size="1.778" layer="27" font="vector" ratio="10" rot="R90" display="off"/>
 </element>
-<element name="CON2" library="SPCoast" package="RJ25-PANEL" value="" x="4.445" y="25.4" rot="R270">
+<element name="CON2" library="SPCoast" package="RJ25-PANEL" value="RJ12/6" x="4.445" y="25.4" rot="R270">
 <attribute name="AMP" value="520250-3" x="4.445" y="25.4" size="1.778" layer="27" font="vector" ratio="10" rot="R270" display="off"/>
 <attribute name="OPL" value="none" x="4.445" y="25.4" size="1.778" layer="27" font="vector" ratio="10" rot="R270" display="off"/>

Commit message: normalized values
Parts:
- BOARD1: value BOARD50X50-HOHOLES -> BOARD; device SPCoast:BOARD-SEED5X5-NOHOLES -> SPCoast:BOARD-SEEED5X5-NOHOLES
- U$1: value OSHW-LOGOM -> OSHW
Changed lines of the file:
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@@
 </autorouter>
 <elements>
-<element name="U$1" library="SparkFun" package="OSHW-LOGO-M" value="OSHW-LOGOM" x="43.18" y="42.926"/>
+<element name="U$1" library="SparkFun" package="OSHW-LOGO-M" value="OSHW" x="43.18" y="42.926"/>
 <element name="J3" library="SPCoast" package="1X06_LOCK" value="0.100" x="31.75" y="6.35" smashed="yes" rot="R180">
 <attribute name="NAME" x="27.94" y="-0.508" size="1.27" layer="25" font="vector" rot="R180"/>
 <attribute name="VALUE" x="33.02" y="9.652" size="1.27" layer="27" font="vector" rot="R180"/>
 </element>
-<element name="BOARD1" library="SPCoast" package="BOARD-SEED5X5-NOHOLES" value="BOARD50X50-HOHOLES" x="0" y="0"/>
+<element name="BOARD1" library="SPCoast" package="BOARD-SEEED5X5-NOHOLES" value="BOARD" x="0" y="0"/>
 <element name="V+" library="SPCoast" package="1X02_LOCK" value="0.100" x="41.91" y="6.35" smashed="yes" rot="R90">
 <attribute name="NAME" x="43.0022" y="12.6492" size="1.27" layer="25" ratio="10" rot="R180"/>
